File: FeriNixie 12-Tube ClocKalc.kicad_pcb (KiCad board)
At the start: 4 copper layers, 534 parts, among them J1 C2765186, Q1 C22392287, Q10 C22392287, Q100 C22392287, Q101 C22392287, Q102 C22392287, Q103 C22392287, Q104 C22392287, Q105 C22392287, Q106 C22392287, Q107 C22392287, Q108 C22392287, Q109 C22392287, Q11 C22392287, Q110 C22392287, Q111 C22392287, Q112 C22392287, Q113 C22392287, Q114 C22392287, Q115 C22392287, Q116 C22392287, Q117 C22392287, Q118 C22392287, Q119 C22392287, Q12 C22392287, Q120 C22392287, Q121 C22392287, Q122 C22392287, Q123 C22392287, Q124 C22392287, Q125 C22392287, Q126 C22392287, Q127 C22392287, Q128 C22392287, Q129 C22392287, Q13 C22392287, Q130 C22392287, Q131 C22392287, Q132 C22392287, Q133 C22392287, Q134 C22392287, Q135 C22392287, Q136 C22392287, Q137 C22392287, Q138 C22392287, Q139 C22392287, Q14 C22392287, Q140 C22392287, Q141 C22392287, Q142 C22392287, Q143 C22392287, Q144 C22392287, Q15 C22392287, Q16 C22392287, Q17 C22392287, Q18 C22392287, Q19 C22392287, Q2 C22392287, Q20 C22392287, Q21 C22392287, Q22 C22392287, Q23 C22392287, Q24 C22392287, Q25 C22392287, Q26 C22392287, Q27 C22392287, Q28 C22392287, Q29 C22392287, Q3 C22392287, Q30 C22392287, Q31 C22392287, Q32 C22392287, Q33 C22392287, Q34 C22392287, Q35 C22392287, Q36 C22392287, Q37 C22392287, Q38 C22392287, Q39 C22392287, Q4 C22392287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

Commit message: Tooooons of changes... stupid amount of changes
Parts:
- removed R260, R261, R264, R265, R266: 120, Resistor_SMD:R_0402_1005Metric
- added D6: C42407105, Diode_SMD:D_0402_1005Metric, F.Cu at (50.5, 76.5)
- added F1: C354900, Capacitor_THT:C_Disc_D10.5mm_W5.0mm_P5.00mm, F.Cu at (49.5, 55.0)
- added NE1: Voltage Indicator, FeriNixie:NeonIndicator_2ML_1MH_B10A, F.Cu at (301.6, 137.2)
- added NE2: ~, FeriNixie:NeonIndicator_2ML_1MH_B10A, F.Cu at (301.6, 139.8)
- added NE3: Run, FeriNixie:NeonIndicator_A1B_A1C, F.Cu at (299.1, 150.8)
- added NE4: BLOWN, FeriNixie:NeonIndicator_A1B_A1C, F.Cu at (299.1, 153.8)
- added REF**: PinHeader_1x01_P2.54mm_Vertical, Connector_PinHeader_2.54mm:PinHeader_1x01_P2.54mm_Vertical, F.Cu at (43.5, 55.0)
- added REF**: MountingHole_2.2mm_M2, MountingHole:MountingHole_2.2mm_M2, F.Cu at (149.5, 38.0)
- added REF**: MountingHole_2.2mm_M2, MountingHole:MountingHole_2.2mm_M2, F.Cu at (255.0, 38.0)
- added REF**: PinHeader_1x01_P2.54mm_Vertical, Connector_PinHeader_2.54mm:PinHeader_1x01_P2.54mm_Vertical, F.Cu at (43.5, 59.5)
- added REF**: MountingHole_2.2mm_M2, MountingHole:MountingHole_2.2mm_M2, F.Cu at (44.0, 38.0)
- added SW3: C309069, NixFootprints:SW_SPST_SS11-BBIWG-R20-R, F.Cu at (57.5, 44.0)
- added U46: GAQY214DE_DEH, Package_DIP:SMDIP-4_W7.62mm, F.Cu at (293.7, 139.3)
- added U47: GAQY214DE_DEH, Package_DIP:SMDIP-4_W7.62mm, F.Cu at (293.5, 145.0)
- R255, R256: value 10K -> 200K; footprint Resistor_SMD:R_0402_1005Metric -> Resistor_SMD:R_1206_3216Metric
- R257, R259: value 120 -> 330; footprint Resistor_SMD:R_0402_1005Metric -> Resistor_SMD:R_1206_3216Metric
- R262: value 120 -> 100K; footprint Resistor_SMD:R_0402_1005Metric -> Resistor_SMD:R_1206_3216Metric
- R263: value 21K -> 100K; footprint Resistor_SMD:R_0402_1005Metric -> Resistor_SMD:R_1206_3216Metric
- SW1, SW2: footprint Button_Switch_SMD:SW_Push_1P1T_NO_CK_KMR2 -> NixFootprints:PB_SPST_GT-TZ084B-H015-L1
- moved U25 280.8 mm to (71.0, 136.0), turned to 90 degrees
- moved R254 280.3 mm to (67.0, 136.5), turned to 90 degrees
- moved R243 277.1 mm to (69.3, 132.8), turned to -90 degrees
- moved R225 272.4 mm to (70.8, 132.8), turned to -90 degrees
- moved U26 271.0 mm to (81.5, 136.0), turned to 90 degrees
- moved R248 268.8 mm to (79.3, 133.7)
- moved D1 268.4 mm to (50.5, 71.7), turned to -90 degrees
- moved R208 267.9 mm to (72.5, 132.8), turned to -90 degrees
- moved R230 265.3 mm to (79.8, 132.5)
- moved U27 264.7 mm to (88.5, 136.0), turned to 90 degrees
- moved R213 259.5 mm to (82.8, 132.0), turned to -90 degrees
- moved R241 258.7 mm to (87.3, 132.8), turned to -90 degrees
- moved U28 255.1 mm to (99.0, 136.0), turned to 90 degrees
- moved R223 254.3 mm to (88.5, 132.8), turned to -90 degrees
- moved R244 249.9 mm to (97.2, 132.8), turned to -90 degrees
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Connections:
- C19 pad 1: Net-(U25-VCC) -> +5V
- C19 pad 2: +5V -> GND
- C20 pad 1: Net-(U26-VCC) -> +5V
- C20 pad 2: +5V -> GND
- C21 pad 1: Net-(U27-VCC) -> +5V
- C21 pad 2: +5V -> GND
- C22 pad 1: Net-(U28-VCC) -> +5V
- C22 pad 2: +5V -> GND
- C23 pad 1: Net-(U29-VCC) -> +5V
- C23 pad 2: +5V -> GND
- C24 pad 1: Net-(U30-VCC) -> +5V
- C24 pad 2: +5V -> GND
- C25 pad 1: Net-(U31-VCC) -> +5V
- C25 pad 2: +5V -> GND
- C26 pad 1: Net-(U32-VCC) -> +5V
- C26 pad 2: +5V -> GND
- C27 pad 1: Net-(U33-VCC) -> +5V
- C27 pad 2: +5V -> GND
- C28 pad 1: Net-(U34-VCC) -> +5V
- C28 pad 2: +5V -> GND
- C29 pad 1: Net-(U35-VCC) -> +5V
- C29 pad 2: +5V -> GND
- C30 pad 1: Net-(U36-VCC) -> +5V
- C30 pad 2: +5V -> GND
- C31 pad 1: Net-(U37-VCC) -> +5V
- C31 pad 2: +5V -> GND
- C32 pad 1: Net-(U38-VCC) -> +5V
- C32 pad 2: +5V -> GND
- C33 pad 1: Net-(U39-VCC) -> +5V
- C33 pad 2: +5V -> GND
- C34 pad 1: Net-(U40-VCC) -> +5V
- C34 pad 2: +5V -> GND
- C35 pad 1: Net-(U41-VCC) -> +5V
- C35 pad 2: +5V -> GND
- C36 pad 1: Net-(U42-VCC) -> +5V
- C36 pad 2: +5V -> GND
- D1 pad 2: VAC -> POW
- PS1 pad 2: VAC -> POW
- PS2 pad 2: VAC -> POW
- R204 pad 1: Net-(D6-A) -> Net-(D5-A)
- R206 pad 1: Net-(D10-A) -> Net-(D5-A)
- R207 pad 1: Net-(D10-A) -> Net-(D5-A)
- R208 pad 1: Net-(D10-A) -> Net-(D5-A)
- R209 pad 1: Net-(D10-A) -> Net-(D5-A)
- R210 pad 1: Net-(D10-A) -> Net-(D5-A)
- R211 pad 1: Net-(D6-A) -> Net-(D5-A)
- R212 pad 1: Net-(D6-A) -> Net-(D5-A)
- R213 pad 1: Net-(D10-A) -> Net-(D5-A)
- R214 pad 1: Net-(D6-A) -> Net-(D5-A)
- R215 pad 1: Net-(D6-A) -> Net-(D5-A)
- R216 pad 1: Net-(D6-A) -> Net-(D5-A)
- R221 pad 1: Net-(D7-A) -> Net-(D4-A)
- R223 pad 1: Net-(D11-A) -> Net-(D4-A)
- R224 pad 1: Net-(D11-A) -> Net-(D4-A)
- R225 pad 1: Net-(D11-A) -> Net-(D4-A)
- R226 pad 1: Net-(D11-A) -> Net-(D4-A)
- R227 pad 1: Net-(D11-A) -> Net-(D4-A)
- R228 pad 1: Net-(D7-A) -> Net-(D4-A)
- R229 pad 1: Net-(D7-A) -> Net-(D4-A)
- R230 pad 1: Net-(D11-A) -> Net-(D4-A)
- R231 pad 1: Net-(D7-A) -> Net-(D4-A)
- R232 pad 1: Net-(D7-A) -> Net-(D4-A)
- R233 pad 1: Net-(D7-A) -> Net-(D4-A)
- R239 pad 1: Net-(D8-A) -> Net-(D3-A)
- R241 pad 1: Net-(D12-A) -> Net-(D3-A)
- R242 pad 1: Net-(D12-A) -> Net-(D3-A)
- R243 pad 1: Net-(D12-A) -> Net-(D3-A)
- R244 pad 1: Net-(D12-A) -> Net-(D3-A)
- R245 pad 1: Net-(D12-A) -> Net-(D3-A)
- R246 pad 1: Net-(D8-A) -> Net-(D3-A)
- R247 pad 1: Net-(D8-A) -> Net-(D3-A)
- R248 pad 1: Net-(D12-A) -> Net-(D3-A)
- R249 pad 1: Net-(D8-A) -> Net-(D3-A)
- R250 pad 1: Net-(D8-A) -> Net-(D3-A)
- R251 pad 1: Net-(D8-A) -> Net-(D3-A)
- R254 pad 1: Net-(D13-A) -> Net-(D2-A)
- R255 pad 1: Net-(D9-A) -> VAC
- R255 pad 2: Net-(U31-SER) -> Net-(NE1-A)
- R256 pad 1: Net-(D2-A) -> Net-(R256-Pad1)
- R256 pad 2: Net-(U37-SER) -> Net-(NE2-A)
- R257 pad 1: Net-(D6-K) -> Net-(U45-GPIO21)
- R257 pad 2: GND -> Net-(R257-Pad2)
- R259 pad 1: Net-(D7-K) -> Net-(U45-GPIO20)
- R259 pad 2: GND -> Net-(R259-Pad2)
- R262 pad 1: Net-(D10-K) -> Net-(R262-Pad1)
- R262 pad 2: GND -> Net-(NE3-A)
- R263 pad 1: /RESET_BTN -> Net-(SW3-A)
- R263 pad 2: Net-(R263-Pad2) -> Net-(NE4-A)
- SW2 pad 2: Net-(R263-Pad2) -> /RESET_BTN
- U25 pad 16: Net-(U25-VCC) -> +5V
- U26 pad 16: Net-(U26-VCC) -> +5V
- U27 pad 16: Net-(U27-VCC) -> +5V
- U28 pad 16: Net-(U28-VCC) -> +5V
- U29 pad 16: Net-(U29-VCC) -> +5V
- U30 pad 16: Net-(U30-VCC) -> +5V
- U30 pad 9: unconnected-(U30-QH'-Pad9) -> Net-(U30-QH')
- U31 pad 14: Net-(U31-SER) -> Net-(U30-QH')
- U31 pad 16: Net-(U31-VCC) -> +5V
- U32 pad 16: Net-(U32-VCC) -> +5V
- U33 pad 16: Net-(U33-VCC) -> +5V
- U34 pad 16: Net-(U34-VCC) -> +5V
- U35 pad 16: Net-(U35-VCC) -> +5V
- U36 pad 16: Net-(U36-VCC) -> +5V
- U36 pad 9: unconnected-(U36-QH'-Pad9) -> Net-(U36-QH')
- U37 pad 14: Net-(U37-SER) -> Net-(U36-QH')
- U37 pad 16: Net-(U37-VCC) -> +5V
- U38 pad 16: Net-(U38-VCC) -> +5V
- U39 pad 16: Net-(U39-VCC) -> +5V
- U40 pad 16: Net-(U40-VCC) -> +5V
- U41 pad 16: Net-(U41-VCC) -> +5V
- U42 pad 16: Net-(U42-VCC) -> +5V
- U45 pad 17: Net-(D13-A) -> unconnected-(U45-GPIO14-Pad17)
- U45 pad 18: Net-(D12-A) -> unconnected-(U45-GPIO15-Pad18)
- U45 pad 27: Net-(D11-A) -> unconnected-(U45-GPIO16-Pad27)
- U45 pad 28: Net-(D10-A) -> unconnected-(U45-GPIO17-Pad28)
- U45 pad 29: Net-(D9-A) -> unconnected-(U45-GPIO18-Pad29)
- U45 pad 30: Net-(D8-A) -> unconnected-(U45-GPIO19-Pad30)
- U45 pad 31: Net-(D7-A) -> Net-(U45-GPIO20)
- U45 pad 32: Net-(D6-A) -> Net-(U45-GPIO21)
Routing:
- net GND: track 0.00 -> 1050.6 mm, vias 0 -> 98
- net +5V: track 0.00 -> 598.4 mm, vias 0 -> 45
- net ISO_5V: track 0.00 -> 335.9 mm, vias 0 -> 24
- net VCOM: track 0.00 -> 287.5 mm
- net POW: track 0.00 -> 268.4 mm, vias 0 -> 1
- net ISO_GND: track 1110.4 -> 1342.4 mm, vias 24 -> 48
- net Net-(D3-A): track 0.00 -> 228.9 mm, vias 0 -> 21
- net Net-(D5-A): track 0.00 -> 226.4 mm, vias 0 -> 19
- net Net-(D4-A): track 0.00 -> 225.0 mm, vias 0 -> 21
- net Net-(D2-A): track 0.00 -> 200.0 mm, vias 0 -> 2
- net +3V3: track 0.00 -> 43.0 mm
- net +170V: track 208.9 -> 235.6 mm, vias 0 -> 2
- net Net-(U16-INC): track 0.00 -> 24.6 mm, vias 0 -> 2
- net Net-(U14-INC): track 0.00 -> 24.6 mm, vias 0 -> 2
- net Net-(U18-INC): track 0.00 -> 24.6 mm, vias 0 -> 2
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- added copper zone on B.Cu, net GND
- added copper zone on F.Cu, net GND
- added copper zone on In1.Cu, net GND
- added copper zone on In2.Cu, net GND
- added copper zone on B.Cu, net ISO_GND
- added copper zone on In1.Cu, net ISO_GND
- added copper zone on In2.Cu, net ISO_GND
Other:
- board outline added: 217 x 115.5 mm

Commit message: changes
Parts:
- removed D10, D11, D12, D13, D7, D8, D9: C5355434, LED_SMD:LED_0603_1608Metric
- removed the D6 at (291.6, 162.3)
- added REF**: MountingHole_2.2mm_M2, MountingHole:MountingHole_2.2mm_M2, F.Cu at (44.0, 147.5)
- added REF**: MountingHole_2.2mm_M2, MountingHole:MountingHole_2.2mm_M2, F.Cu at (149.5, 147.5)
- added REF**: MountingHole_2.2mm_M2, MountingHole:MountingHole_2.2mm_M2, F.Cu at (255.0, 147.5)
- moved NE1 273.9 mm to (44.0, 44.0)
- moved NE4 268.9 mm to (44.9, 66.2), turned to 90 degrees
- moved R255 258.0 mm to (43.0, 48.9), turned to 90 degrees
- moved R263 254.0 mm to (44.9, 72.1), turned to 90 degrees
- moved C13 212.6 mm to (61.8, 114.0), turned to -90 degrees
- moved C19 203.4 mm to (68.0, 140.4), turned to -90 degrees
- moved C20 193.5 mm to (78.5, 140.4), turned to -90 degrees
- moved C21 187.1 mm to (85.5, 140.4), turned to -90 degrees
- moved C22 177.0 mm to (96.0, 140.4), turned to -90 degrees
- moved C23 166.9 mm to (106.5, 140.4), turned to -90 degrees
- moved C24 160.4 mm to (113.5, 140.4), turned to -90 degrees
- moved C25 150.6 mm to (124.0, 140.4), turned to -90 degrees
- moved C26 140.8 mm to (134.5, 140.4), turned to -90 degrees
- moved C27 134.6 mm to (141.5, 140.4), turned to -90 degrees
- moved C28 125.1 mm to (152.0, 140.5), turned to -90 degrees
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Connections:
- D2 pad 1: Net-(D2-K) -> GND
- D3 pad 1: Net-(D3-K) -> GND
- D4 pad 1: Net-(D4-K) -> GND
- D5 pad 1: Net-(D5-K) -> GND
- R196 pad 1: Net-(D2-K) -> Net-(U45-GPIO22)
- R196 pad 2: GND -> Net-(D2-A)
- R197 pad 1: Net-(D3-K) -> Net-(U45-GPIO23)
- R197 pad 2: GND -> Net-(D3-A)
- R198 pad 1: Net-(D4-K) -> Net-(U45-GPIO24)
- R198 pad 2: GND -> Net-(D4-A)
- R199 pad 1: Net-(D5-K) -> Net-(U45-GPIO25)
- R199 pad 2: GND -> Net-(D5-A)
- R200 pad 1: Net-(D5-A) -> Net-(U45-GPIO25)
- R201 pad 1: Net-(D5-A) -> Net-(U45-GPIO25)
- R202 pad 1: Net-(D5-A) -> Net-(U45-GPIO25)
- R203 pad 1: Net-(D5-A) -> Net-(U45-GPIO25)
- R204 pad 1: Net-(D5-A) -> Net-(U45-GPIO25)
- R205 pad 1: Net-(D5-A) -> Net-(U45-GPIO25)
- R206 pad 1: Net-(D5-A) -> Net-(U45-GPIO25)
- R207 pad 1: Net-(D5-A) -> Net-(U45-GPIO25)
- R208 pad 1: Net-(D5-A) -> Net-(U45-GPIO25)
- R209 pad 1: Net-(D5-A) -> Net-(U45-GPIO25)
- R210 pad 1: Net-(D5-A) -> Net-(U45-GPIO25)
- R211 pad 1: Net-(D5-A) -> Net-(U45-GPIO25)
- R212 pad 1: Net-(D5-A) -> Net-(U45-GPIO25)
- R213 pad 1: Net-(D5-A) -> Net-(U45-GPIO25)
- R214 pad 1: Net-(D5-A) -> Net-(U45-GPIO25)
- R215 pad 1: Net-(D5-A) -> Net-(U45-GPIO25)
- R216 pad 1: Net-(D5-A) -> Net-(U45-GPIO25)
- R217 pad 1: Net-(D4-A) -> Net-(U45-GPIO24)
- R218 pad 1: Net-(D4-A) -> Net-(U45-GPIO24)
- R219 pad 1: Net-(D4-A) -> Net-(U45-GPIO24)
- R220 pad 1: Net-(D4-A) -> Net-(U45-GPIO24)
- R221 pad 1: Net-(D4-A) -> Net-(U45-GPIO24)
- R222 pad 1: Net-(D4-A) -> Net-(U45-GPIO24)
- R223 pad 1: Net-(D4-A) -> Net-(U45-GPIO24)
- R224 pad 1: Net-(D4-A) -> Net-(U45-GPIO24)
- R225 pad 1: Net-(D4-A) -> Net-(U45-GPIO24)
- R226 pad 1: Net-(D4-A) -> Net-(U45-GPIO24)
- R227 pad 1: Net-(D4-A) -> Net-(U45-GPIO24)
- R228 pad 1: Net-(D4-A) -> Net-(U45-GPIO24)
- R229 pad 1: Net-(D4-A) -> Net-(U45-GPIO24)
- R230 pad 1: Net-(D4-A) -> Net-(U45-GPIO24)
- R231 pad 1: Net-(D4-A) -> Net-(U45-GPIO24)
- R232 pad 1: Net-(D4-A) -> Net-(U45-GPIO24)
- R233 pad 1: Net-(D4-A) -> Net-(U45-GPIO24)
- R234 pad 1: Net-(D5-A) -> Net-(U45-GPIO25)
- R235 pad 1: Net-(D3-A) -> Net-(U45-GPIO23)
- R236 pad 1: Net-(D3-A) -> Net-(U45-GPIO23)
- R237 pad 1: Net-(D3-A) -> Net-(U45-GPIO23)
- R238 pad 1: Net-(D3-A) -> Net-(U45-GPIO23)
- R239 pad 1: Net-(D3-A) -> Net-(U45-GPIO23)
- R240 pad 1: Net-(D3-A) -> Net-(U45-GPIO23)
- R241 pad 1: Net-(D3-A) -> Net-(U45-GPIO23)
- R242 pad 1: Net-(D3-A) -> Net-(U45-GPIO23)
- R243 pad 1: Net-(D3-A) -> Net-(U45-GPIO23)
- R244 pad 1: Net-(D3-A) -> Net-(U45-GPIO23)
- R245 pad 1: Net-(D3-A) -> Net-(U45-GPIO23)
- R246 pad 1: Net-(D3-A) -> Net-(U45-GPIO23)
- R247 pad 1: Net-(D3-A) -> Net-(U45-GPIO23)
- R248 pad 1: Net-(D3-A) -> Net-(U45-GPIO23)
- R249 pad 1: Net-(D3-A) -> Net-(U45-GPIO23)
- R250 pad 1: Net-(D3-A) -> Net-(U45-GPIO23)
- R251 pad 1: Net-(D3-A) -> Net-(U45-GPIO23)
- R252 pad 1: Net-(D4-A) -> Net-(U45-GPIO24)
- R253 pad 1: Net-(D3-A) -> Net-(U45-GPIO23)
- R254 pad 1: Net-(D2-A) -> Net-(U45-GPIO22)
- U45 pad 34: Net-(D2-A) -> Net-(U45-GPIO22)
- U45 pad 35: Net-(D3-A) -> Net-(U45-GPIO23)
- U45 pad 36: Net-(D4-A) -> Net-(U45-GPIO24)
- U45 pad 37: Net-(D5-A) -> Net-(U45-GPIO25)
Routing:
- net GND: track 1050.6 -> 1310.2 mm, vias 98 -> 103
- net Net-(U45-GPIO23): track 0.00 -> 230.5 mm, vias 0 -> 21
- net Net-(U45-GPIO25): track 0.00 -> 227.3 mm, vias 0 -> 19
- net Net-(D3-A): track 228.9 -> 1.92 mm, vias 21 -> 0
- net Net-(U45-GPIO24): track 0.00 -> 226.0 mm, vias 0 -> 21
- net Net-(D5-A): track 226.4 -> 1.50 mm, vias 19 -> 0
- net Net-(D4-A): track 225.0 -> 1.71 mm, vias 21 -> 0
- net Net-(U45-GPIO22): track 0.00 -> 201.0 mm, vias 0 -> 2
- net Net-(D2-A): track 200.0 -> 2.12 mm, vias 2 -> 0
- net Net-(U45-GPIO21): track 0.00 -> 125.9 mm, vias 0 -> 5
- net Net-(U45-GPIO20): track 0.00 -> 88.9 mm, vias 0 -> 2
- net VCOM: track 287.5 -> 333.4 mm
- net Net-(SW3-A): track 11.6 -> 35.8 mm, vias 0 -> 1
- net Net-(R258-Pad2): track 0.00 -> 21.7 mm
- net POW: track 268.4 -> 283.7 mm
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Other:
- board text added: "BOOT"
- board text added: "RCK"
- board text added: "RESET"
- board text added: "SCK"
- board text added: "SER"
- board text added: "~{CLR}"
