File: FeriNixie 12-Tube ClocKalc.kicad_pcb (KiCad board)
At the start: 4 copper layers, 217 x 115.5 mm, 553 parts, among them J1 Conn_01x02_Socket, Q1 C22392287, Q10 C22392287, Q100 C22392287, Q101 C22392287, Q102 C22392287, Q103 C22392287, Q104 C22392287, Q105 C22392287, Q106 C22392287, Q107 C22392287, Q108 C22392287, Q109 C22392287, Q11 C22392287, Q110 C22392287, Q111 C22392287, Q112 C22392287, Q113 C22392287, Q114 C22392287, Q115 C22392287, Q116 C22392287, Q117 C22392287, Q118 C22392287, Q119 C22392287, Q12 C22392287, Q120 C22392287, Q121 C22392287, Q122 C22392287, Q123 C22392287, Q124 C22392287, Q125 C22392287, Q126 C22392287, Q127 C22392287, Q128 C22392287, Q129 C22392287, Q13 C22392287, Q130 C22392287, Q131 C22392287, Q132 C22392287, Q133 C22392287, Q134 C22392287, Q135 C22392287, Q136 C22392287, Q137 C22392287, Q138 C22392287, Q139 C22392287, Q14 C22392287, Q140 C22392287, Q141 C22392287, Q142 C22392287, Q143 C22392287, Q144 C22392287, Q15 C22392287, Q16 C22392287, Q17 C22392287, Q18 C22392287, Q19 C22392287, Q2 C22392287, Q20 C22392287, Q21 C22392287, Q22 C22392287, Q23 C22392287, Q24 C22392287, Q25 C22392287, Q26 C22392287, Q27 C22392287, Q28 C22392287, Q29 C22392287, Q3 C22392287, Q30 C22392287, Q31 C22392287, Q32 C22392287, Q33 C22392287, Q34 C22392287, Q35 C22392287, Q36 C22392287, Q37 C22392287, Q38 C22392287, Q39 C22392287, Q4 C22392287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

Commit message: Final changes before printing
Parts:
- removed C49, C50: 15pF, Capacitor_SMD:C_0402_1005Metric
- removed TXAL1: Q13FC1350000400, JLCPCB_Imported:FC-135R_L3.2-W1.5
Connections:
- R266 pad 2: /FLIP_32kHz -> /D_GPIO-6
- R273 pad 2: /FLIP_32kHz -> /D_GPIO-6
Routing:
- net /D_GPIO-6: track 0.00 -> 30.0 mm, vias 0 -> 2
- net GND: track 1365.8 -> 1358.6 mm, vias 150 -> 149
- net +3V3: track 64.9 -> 59.3 mm, vias 5 -> 3
- net /FLIP_32kHz: track 4.94 -> 0.00 mm
- net +5V: track 615.2 -> 614.0 mm, vias 39 -> 38
- net +170V: track 304.5 -> 305.5 mm
- net VCOM: track 139.8 -> 138.9 mm
- net Net-(U36-B): track 62.0 -> 62.8 mm
Other:
- board text added: "FeriNixie 12-Tube ClocKalc One of one, custom display for a calculator / clock combination device 120Vac Mains input RP2040 Driver with USB C 12x B-16851453 Burroughs Nixies"
- board text added: "Github"
- board text added: "UwU"
- board text removed: "FeriNixie 12-Tube ClocKalc One of one, custom display"
