File: FeriNixie 12-Tube ClocKalc.kicad_pcb (KiCad board)
At the start: 4 copper layers, 217 x 115.5 mm, 550 parts, among them J1 Conn_01x02_Socket, Q1 C22392287, Q10 C22392287, Q100 C22392287, Q101 C22392287, Q102 C22392287, Q103 C22392287, Q104 C22392287, Q105 C22392287, Q106 C22392287, Q107 C22392287, Q108 C22392287, Q109 C22392287, Q11 C22392287, Q110 C22392287, Q111 C22392287, Q112 C22392287, Q113 C22392287, Q114 C22392287, Q115 C22392287, Q116 C22392287, Q117 C22392287, Q118 C22392287, Q119 C22392287, Q12 C22392287, Q120 C22392287, Q121 C22392287, Q122 C22392287, Q123 C22392287, Q124 C22392287, Q125 C22392287, Q126 C22392287, Q127 C22392287, Q128 C22392287, Q129 C22392287, Q13 C22392287, Q130 C22392287, Q131 C22392287, Q132 C22392287, Q133 C22392287, Q134 C22392287, Q135 C22392287, Q136 C22392287, Q137 C22392287, Q138 C22392287, Q139 C22392287, Q14 C22392287, Q140 C22392287, Q141 C22392287, Q142 C22392287, Q143 C22392287, Q144 C22392287, Q15 C22392287, Q16 C22392287, Q17 C22392287, Q18 C22392287, Q19 C22392287, Q2 C22392287, Q20 C22392287, Q21 C22392287, Q22 C22392287, Q23 C22392287, Q24 C22392287, Q25 C22392287, Q26 C22392287, Q27 C22392287, Q28 C22392287, Q29 C22392287, Q3 C22392287, Q30 C22392287, Q31 C22392287, Q32 C22392287, Q33 C22392287, Q34 C22392287, Q35 C22392287, Q36 C22392287, Q37 C22392287, Q38 C22392287, Q39 C22392287, Q4 C22392287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

Commit message: Update FeriNixie 12-Tube ClocKalc.kicad_pcb
Parts:
- added REF**: PinHeader_1x06_P2.54mm_Vertical, Connector_PinHeader_2.54mm:PinHeader_1x06_P2.54mm_Vertical, F.Cu at (227.5, 149.0)
- added REF**: PinHeader_1x06_P2.54mm_Vertical, Connector_PinHeader_2.54mm:PinHeader_1x06_P2.54mm_Vertical, F.Cu at (207.1, 149.0)
- added REF**: PinHeader_1x02_P2.54mm_Vertical, Connector_PinHeader_2.54mm:PinHeader_1x02_P2.54mm_Vertical, F.Cu at (198.6, 149.0)
Routing:
- net /D_GPIO-14: track 0.00 -> 32.8 mm, vias 0 -> 1
- net /D_GPIO-15: track 0.00 -> 31.0 mm, vias 0 -> 1
- net /D_GPIO-16: track 0.00 -> 27.4 mm, vias 0 -> 2
- net /D_GPIO-17: track 0.00 -> 23.1 mm, vias 0 -> 1
- net /D_GPIO-18: track 0.00 -> 20.7 mm, vias 0 -> 1
- net /D_GPIO-19: track 0.00 -> 19.0 mm, vias 0 -> 1
- net +5V: track 614.0 -> 630.0 mm
- net /D_GPIO-20: track 0.00 -> 13.2 mm, vias 0 -> 1
- net /D_GPIO-21: track 0.00 -> 11.8 mm, vias 0 -> 1
- net /D_GPIO-22: track 0.00 -> 10.4 mm, vias 0 -> 1
- net /D_GPIO-23: track 0.00 -> 7.91 mm, vias 0 -> 1
- net /D_GPIO-25: track 0.00 -> 7.62 mm, vias 0 -> 1
- net /D_GPIO-24: track 0.00 -> 7.19 mm, vias 0 -> 1
- net /BOOT: track 39.9 -> 40.7 mm
- net GND: vias 149 -> 153
Other:
- board text added: "+5V"
- board text added: "19"
- board text added: "20"
- board text added: "25"
- board text added: "GND"
