File: FeriNixie 12-Tube ClocKalc.kicad_sch (KiCad schematic)
At the start: 510 parts, among them J1 C2765186, Q1 C22392287, Q10 C22392287, Q100 C22392287, Q101 C22392287, Q102 C22392287, Q103 C22392287, Q104 C22392287, Q105 C22392287, Q106 C22392287, Q107 C22392287, Q108 C22392287, Q109 C22392287, Q11 C22392287, Q110 C22392287, Q111 C22392287, Q112 C22392287, Q113 C22392287, Q114 C22392287, Q115 C22392287, Q116 C22392287, Q117 C22392287, Q118 C22392287, Q119 C22392287, Q12 C22392287, Q120 C22392287, Q121 C22392287, Q122 C22392287, Q123 C22392287, Q124 C22392287, Q125 C22392287, Q126 C22392287, Q127 C22392287, Q128 C22392287, Q129 C22392287, Q13 C22392287, Q130 C22392287, Q131 C22392287, Q132 C22392287, Q133 C22392287, Q134 C22392287, Q135 C22392287, Q136 C22392287, Q137 C22392287, Q138 C22392287, Q139 C22392287, Q14 C22392287, Q140 C22392287, Q141 C22392287, Q142 C22392287, Q143 C22392287, Q144 C22392287, Q15 C22392287, Q16 C22392287, Q17 C22392287, Q18 C22392287, Q19 C22392287, Q2 C22392287, Q20 C22392287, Q21 C22392287, Q22 C22392287, Q23 C22392287, Q24 C22392287, Q25 C22392287, Q26 C22392287, Q27 C22392287, Q28 C22392287, Q29 C22392287, Q3 C22392287, Q30 C22392287, Q31 C22392287, Q32 C22392287, Q33 C22392287, Q34 C22392287, Q35 C22392287, Q36 C22392287, Q37 C22392287, Q38 C22392287, Q39 C22392287, Q4 C22392287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

Commit message: Tooooons of changes... stupid amount of changes
Parts:
- added D6: C42407105, Diode_SMD:D_0402_1005Metric, symbol Device:D_TVS
- added F1: C354900, Capacitor_THT:C_Disc_D10.5mm_W5.0mm_P5.00mm, symbol Device:Fuse
- added NE1: Voltage Indicator, FeriNixie:NeonIndicator_2ML_1MH_B10A, symbol FeriNixie:NeonIndicator_2ML_1MH_B10A
- added NE2: (no value), FeriNixie:NeonIndicator_2ML_1MH_B10A, symbol FeriNixie:NeonIndicator_2ML_1MH_B10A
- added NE3: Run, FeriNixie:NeonIndicator_A1B_A1C, symbol FeriNixie:NeonIndicator_A1B_A1C
- added NE4: BLOWN, FeriNixie:NeonIndicator_A1B_A1C, symbol FeriNixie:NeonIndicator_A1B_A1C
- added R255, R256: 200K, Resistor_SMD:R_1206_3216Metric, symbol NixMinis:Mini_R
- added R257, R259: 330, Resistor_SMD:R_1206_3216Metric, symbol NixMinis:Mini_R
- added R262, R263: 100K, Resistor_SMD:R_1206_3216Metric, symbol NixMinis:Mini_R
- added SW3: C309069, NixFootprints:SW_SPST_SS11-BBIWG-R20-R, symbol Switch:SW_SPST
- added U46, U47: GAQY214DE_DEH, Package_DIP:SMDIP-4_W7.62mm, symbol NixSymbols:GAQY214DE_DEH
- SW1, SW2: footprint Button_Switch_SMD:SW_Push_1P1T_NO_CK_KMR2 -> NixFootprints:PB_SPST_GT-TZ084B-H015-L1
Connections:
- net +170V: now also D6.1 (A1)
- net +5V: now also C19.1, C20.1, C21.1, C22.1, C23.1, C24.1, C25.1, C26.1, C27.1, C28.1, C29.1, C30.1, C31.1, C32.1, C33.1, C34.1, C35.1, C36.1, U25.16 (VCC), U26.16 (VCC), U27.16 (VCC), U28.16 (VCC), U29.16 (VCC), U30.16 (VCC), U31.16 (VCC), U32.16 (VCC), U33.16 (VCC), U34.16 (VCC), U35.16 (VCC), U36.16 (VCC), U37.16 (VCC), U38.16 (VCC), U39.16 (VCC), U40.16 (VCC), U41.16 (VCC), U42.16 (VCC); no longer C19.2, C20.2, C21.2, C22.2, C23.2, C24.2, C25.2, C26.2, C27.2, C28.2, C29.2, C30.2, C31.2, C32.2, C33.2, C34.2, C35.2, C36.2
- net GND: now also C19.2, C20.2, C21.2, C22.2, C23.2, C24.2, C25.2, C26.2, C27.2, C28.2, C29.2, C30.2, C31.2, C32.2, C33.2, C34.2, C35.2, C36.2, U46.2, U47.2
- net ISO_GND: now also D6.2 (A2)
- net VAC: now also R255.1, SW3.2 (B); no longer D1.2, PS1.2 (AC/L), PS2.2 (AC/L)
- net VCOM: now also NE1.2 (K), NE2.2 (K), NE3.2 (K)
- net at U45.31 (GPIO20): now also R259.1
- net at U45.32 (GPIO21): now also R257.1
- new net: F1.1, R263.1, SW3.1 (A)
- new net: NE4.1 (A), R263.2
- new net: R257.2, U46.1
- new net: NE3.1 (A), R262.2
- new net: R256.1, U47.4
- new net: NE2.1 (A), R256.2
- new net: R259.2, U47.1
- new net: NE1.1 (A), R255.2
- new net: R262.1, U46.4
- new net POW: D1.2, F1.2, NE4.2 (K), PS1.2 (AC/L), PS2.2 (AC/L), U46.3, U47.3
Other:
- moved on the sheet: D1, J1, NX1, NX10, NX11, NX12, NX2, NX3, NX4, NX5, NX6, NX7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

Commit message: changes
Parts:
- D6: value C42407105 -> C2802304
Connections:
- net GND: now also D2.1 (K), D3.1 (K), D4.1 (K), D5.1 (K); no longer R196.2, R197.2, R198.2, R199.2
- net at R199.1: now also R200.1, R201.1, R202.1, R203.1, R204.1, R205.1, R206.1, R207.1, R208.1, R209.1, R210.1, R211.1, R212.1, R213.1, R214.1, R215.1, R216.1, R234.1, U45.37 (GPIO25); no longer D5.1 (K)
- net at R235.1, R236.1, R237.1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: now also R197.1; no longer D3.2 (A)
- net at R254.1, U45.34 (GPIO22): now also R196.1; no longer D2.2 (A)
- net at R217.1, R218.1, R219.1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: now also R198.1; no longer D4.2 (A)
- new net: D5.2 (A), R199.2
- new net: D3.2 (A), R197.2
- new net: D2.2 (A), R196.2
- new net: D4.2 (A), R198.2

Commit message: Finalize changes for printing
Parts:
- removed C13, C17, C18: 1uF, Capacitor_SMD:C_0402_1005Metric, symbol NixMinis:Mini_C
- removed C15, C16: 15pF, Capacitor_SMD:C_0402_1005Metric, symbol NixMinis:Mini_C
- removed D1: MB6S, Package_TO_SOT_SMD:TO-269AA, symbol Diode_Bridge:MB6S
- removed D2, D3, D4, D5: C5355434, LED_SMD:LED_0603_1608Metric, symbol NixMinis:Mini_D
- removed D6: C2802304, Diode_SMD:D_0402_1005Metric, symbol Device:D_TVS
- removed J1: C2765186, Connector_USB:USB_C_Receptacle_G-Switch_GT-USB-7010ASV, symbol Connector:USB_C_Receptacle_USB2.0_16P
- removed NE3: Run, FeriNixie:NeonIndicator_A1B_A1C, symbol FeriNixie:NeonIndicator_A1B_A1C
- removed PS1, PS2: C22394236, Converter_ACDC:Converter_ACDC_MeanWell_IRM-02-xx_THT, symbol Converter_ACDC:IRM-02-5
- removed R193: 1K, Resistor_SMD:R_0402_1005Metric, symbol NixMinis:Mini_R
- removed R194, R195: 5.1K, Resistor_SMD:R_0402_1005Metric, symbol NixMinis:Mini_R
- removed R262: 100K, Resistor_SMD:R_1206_3216Metric, symbol NixMinis:Mini_R
- removed SW1: BOOT, NixFootprints:PB_SPST_GT-TZ084B-H015-L1, symbol Switch:SW_Push
- removed SW2: RESET, NixFootprints:PB_SPST_GT-TZ084B-H015-L1, symbol Switch:SW_Push
- removed U1, U10, U11, U12, U13, U14, U15, U16, U17, U18, U19, U2, U20, U21, U22, U23, U24, U3, U4, U5, U6, U7, U8, U9: C32713198, Package_SO:JEITA_SOIC-16_3.9x9.9mm_P1.27mm, symbol NixSymbols:CMT8260N0
- removed U25, U26, U27, U28, U29, U30, U31, U32, U33, U34, U35, U36, U37, U38, U39, U40, U41, U42: C53200146, Package_DFN_QFN:QFN-16-1EP_3x3mm_P0.5mm_EP1.45x1.45mm, symbol NixSymbols:74HC595_DHXQFN-16
- removed U43: C7434207, Package_TO_SOT_SMD:TSOT-23-5, symbol NixSymbols:RT9013-33GB
- removed U44: C131025, Package_SO:SOIC-8_5.3x5.3mm_P1.27mm, symbol Memory_Flash:W25Q16JVSS
- removed U45: C2040, Package_DFN_QFN:QFN-56-1EP_7x7mm_P0.4mm_EP3.2x3.2mm, symbol MCU_RaspberryPi:RP2040
- removed U46, U47: GAQY214DE_DEH, Package_DIP:SMDIP-4_W7.62mm, symbol NixSymbols:GAQY214DE_DEH
- removed Y1: C37635394, Crystal:Crystal_SMD_2016-4Pin_2.0x1.6mm, symbol Device:Crystal_GND23
- added C31, C32, C35, C45, C46: 4.7uF, Capacitor_SMD:C_0402_1005Metric, symbol NixMinis:Mini_C
- added C33, C34, C49, C50: 15pF, Capacitor_SMD:C_0402_1005Metric, symbol NixMinis:Mini_C
- added C41, C42, C43, C44, C47, C48: 100nF, Capacitor_SMD:C_0402_1005Metric, symbol NixMinis:Mini_C
- added C51, C52: 100nF, Capacitor_SMD:C_1206_3216Metric, symbol NixMinis:Mini_C
- added D1: SMCJ150CA_C41411757, JLCPCB_Imported:SMC_L6.9-W5.9-LS7.9-BI, symbol JLCPCB_Imported:SMCJ150CA_C41411757
- added J1: Conn_01x02_Socket, Connector_PinSocket_1.00mm:PinSocket_1x02_P1.00mm_Vertical, symbol Connector:Conn_01x02_Socket
- added NE1: Run, FeriNixie:NeonIndicator_A1B_A1C, symbol FeriNixie:NeonIndicator_A1B_A1C
- added R252: 100K, Resistor_SMD:R_1206_3216Metric, symbol NixMinis:Mini_R
- added R254, R260: 5.1K, Resistor_SMD:R_0402_1005Metric, symbol NixMinis:Mini_R
- added R255, R272: 200K, Resistor_SMD:R_1206_3216Metric, symbol NixMinis:Mini_R
- added R261: 1K, Resistor_SMD:R_0402_1005Metric, symbol NixMinis:Mini_R
- added R263: 22K, Resistor_SMD:R_0402_1005Metric, symbol NixMinis:Mini_R
- added R265: 200, Resistor_SMD:R_0402_1005Metric, symbol NixMinis:Mini_R
- added R266, R270, R271, R273, R274, R277, R278: 100, Resistor_SMD:R_0402_1005Metric, symbol NixMinis:Mini_R
- added R275, R276: 10K, Resistor_SMD:R_0402_1005Metric, symbol NixMinis:Mini_R
- added TXAL1: Q13FC1350000400, JLCPCB_Imported:FC-135R_L3.2-W1.5, symbol JLCPCB_Imported:Q13FC1350000400
- added U1, U10, U11, U12, U13, U14, U15, U16, U17, U18, U2, U3, U4, U5, U6, U7, U8, U9: 74HC595D,118, JLCPCB_Imported:SOIC-16_L9.9-W3.9-P1.27-LS6.0-BL, symbol JLCPCB_Imported:74HC595D,118
- added U19, U20, U21, U22, U25: KT-0603R, JLCPCB_Imported:LED-SMD_L1.6-W0.8-R-RD, symbol JLCPCB_Imported:KT-0603R
- added U24: XC6206P332MR, JLCPCB_Imported:SOT-23-3_L2.9-W1.3-P1.90-LS2.4-BR, symbol JLCPCB_Imported:XC6206P332MR
- added U27: TYPE-C_16PIN_2MD(073), JLCPCB_Imported:USB-C-SMD_TYPE-C-16PIN-2MD-073, symbol JLCPCB_Imported:TYPE-C_16PIN_2MD(073)
- added U28: RP2040, JLCPCB_Imported:LQFN-56_L7.0-W7.0-P0.4-EP, symbol JLCPCB_Imported:RP2040
- added U29, U30: TS-1187A-B-A-B, JLCPCB_Imported:SW-SMD_4P-L5.1-W5.1-P3.70-LS6.5-TL_H1.5, symbol JLCPCB_Imported:TS-1187A-B-A-B
- added U31: MB10S_C2488, JLCPCB_Imported:MBS_L4.7-W3.8-P2.40-LS7.0-TL, symbol JLCPCB_Imported:MB10S_C2488
- added U32: IRM-03-5, JLCPCB_Imported:PWRM-TH_IRM-03-5-DIP5, symbol JLCPCB_Imported:IRM-03-5
- added U33: W25Q128JVSIQTR, JLCPCB_Imported:SOIC-8_L5.3-W5.3-P1.27-LS8.0-BL, symbol JLCPCB_Imported:W25Q128JVSIQTR
- added U34, U35, U36, U37, U38, U39, U40, U41: MMBTA42_C20069138, JLCPCB_Imported:SOT-23-3_L2.9-W1.3-P1.90-LS2.4-BR, symbol JLCPCB_Imported:MMBTA42_C20069138
- added X1: X322512MSB4SI, JLCPCB_Imported:CRYSTAL-SMD_4P-L3.2-W2.5-BL, symbol JLCPCB_Imported:X322512MSB4SI
- C37: value 1uF -> 4.7uF
- C38, C39, C40: value 1uF -> 100nF
- F1: now left out of the parts list
- R193: renamed from R196; value 120 -> 560
- R194: renamed from R197; value 120 -> 560
- R195: renamed from R198; value 120 -> 560
- R196: renamed from R199; value 120 -> 560
- R256: value 200K -> 100K
- R257: value 330 -> 22; footprint Resistor_SMD:R_1206_3216Metric -> Resistor_SMD:R_0402_1005Metric
- R258: value 21K -> 22
- R259: value 330 -> 1K; footprint Resistor_SMD:R_1206_3216Metric -> Resistor_SMD:R_0402_1005Metric
- R267: value 27 -> 10K
- R268: value 27 -> 100
- R269: value 200 -> 10K
- SW1: renamed from SW3; footprint NixFootprints:SW_SPST_SS11-BBIWG-R20-R -> JLCPCB_Imported:SW-TH_SS11-BBIWQ-XX
- renumbered C19 to C13, C20 to C14, C21 to C15, C22 to C16, C23 to C17, C24 to C18, C25 to C19, C26 to C20, C27 to C21, C28 to C22, C29 to C23, C30 to C24, C31 to C25, C32 to C26, C33 to C27, C34 to C28, C35 to C29, C36 to C30, C14 to C36, NE1 to NE3, R200 to R197, R201 to R198, R202 to R199, R203 to R200, R204 to R201, R205 to R202, R206 to R203, R207 to R204, R208 to R205, R209 to R206, R210 to R207, R211 to R208, R212 to R209, R213 to R210, R214 to R211, R215 to R212, R216 to R213, R217 to R214, R218 to R215, R219 to R216, R220 to R217, R221 to R218, R222 to R219, R223 to R220, R224 to R221, R225 to R222, R226 to R223, R227 to R224, R228 to R225, R229 to R226, R230 to R227, R231 to R228, R232 to R229, R233 to R230, R234 to R231, R235 to R232, R236 to R233, R237 to R234, R238 to R235, R239 to R236, R240 to R237, R241 to R238, R242 to R239, R243 to R240, R244 to R241, R245 to R242, R246 to R243, R247 to R244, R248 to R245, R249 to R246, R250 to R247, R251 to R248, R252 to R249, R253 to R250, R254 to R251, R255 to R262, R263 to R264
Connections:
- net 1V1 is gone; now on net +3V3: C38.1
- net BOOT_BTN is gone; now on net D-: R258.1
- net ISO_GND is gone; now on net GND: C1.2, C10.2, C11.2, C12.2, C2.2, C3.2, C4.2, C5.2, C6.2, C7.2, C8.2, C9.2, Q1.2 (E), Q10.2 (E), Q100.2 (E), Q101.2 (E), Q102.2 (E), Q103.2 (E), Q104.2 (E), Q105.2 (E), Q106.2 (E), Q107.2 (E), Q108.2 (E), Q109.2 (E), Q11.2 (E), Q110.2 (E), Q111.2 (E), Q112.2 (E), Q113.2 (E), Q114.2 (E), Q115.2 (E), Q116.2 (E), Q117.2 (E), Q118.2 (E), Q119.2 (E), Q12.2 (E), Q120.2 (E), Q121.2 (E), Q122.2 (E), Q123.2 (E), Q124.2 (E), Q125.2 (E), Q126.2 (E), Q127.2 (E), Q128.2 (E), Q129.2 (E), Q13.2 (E), Q130.2 (E), Q131.2 (E), Q132.2 (E), Q133.2 (E), Q134.2 (E), Q135.2 (E), Q136.2 (E), Q137.2 (E), Q138.2 (E), Q139.2 (E), Q14.2 (E), Q140.2 (E), Q141.2 (E), Q142.2 (E), Q143.2 (E), Q144.2 (E), Q15.2 (E), Q16.2 (E), Q17.2 (E), Q18.2 (E), Q19.2 (E), Q2.2 (E), Q20.2 (E), Q21.2 (E), Q22.2 (E), Q23.2 (E), Q24.2 (E), Q25.2 (E), Q26.2 (E), Q27.2 (E), Q28.2 (E), Q29.2 (E), Q3.2 (E), Q30.2 (E), Q31.2 (E), Q32.2 (E), Q33.2 (E), Q34.2 (E), Q35.2 (E), Q36.2 (E), Q37.2 (E), Q38.2 (E), Q39.2 (E), Q4.2 (E), Q40.2 (E), Q41.2 (E), Q42.2 (E), Q43.2 (E), Q44.2 (E), Q45.2 (E), Q46.2 (E), Q47.2 (E), Q48.2 (E), Q49.2 (E), Q5.2 (E), Q50.2 (E), Q51.2 (E), Q52.2 (E), Q53.2 (E), Q54.2 (E), Q55.2 (E), Q56.2 (E), Q57.2 (E), Q58.2 (E), Q59.2 (E), Q6.2 (E), Q60.2 (E), Q61.2 (E), Q62.2 (E), Q63.2 (E), Q64.2 (E), Q65.2 (E), Q66.2 (E), Q67.2 (E), Q68.2 (E), Q69.2 (E), Q7.2 (E), Q70.2 (E), Q71.2 (E), Q72.2 (E), Q73.2 (E), Q74.2 (E), Q75.2 (E), Q76.2 (E), Q77.2 (E), Q78.2 (E), Q79.2 (E), Q8.2 (E), Q80.2 (E), Q81.2 (E), Q82.2 (E), Q83.2 (E), Q84.2 (E), Q85.2 (E), Q86.2 (E), Q87.2 (E), Q88.2 (E), Q89.2 (E), Q9.2 (E), Q90.2 (E), Q91.2 (E), Q92.2 (E), Q93.2 (E), Q94.2 (E), Q95.2 (E), Q96.2 (E), Q97.2 (E), Q98.2 (E), Q99.2 (E)
- net +170V: now also R256.1, C51.2, C52.2, D1.2, R252.1, R255.2, R272.2, U31.1 (+)
- net +3V3: now also C40.1, C31.2, C35.2, C41.1, C42.1, C43.1, C44.1, C45.1, C49.1, R265.1, TXAL1.1, U24.2 (Vout), U28.1 (IOVDD), U28.10 (IOVDD), U28.22 (IOVDD), U28.33 (IOVDD), U28.42 (IOVDD), U28.44 (VREG_IN), U28.48 (USB_VDD), U28.49 (IOVDD), U33.8 (VCC); no longer C37.1, R269.1
- net +5V: now also C32.2, U1.16 (VCC), U10.16 (VCC), U11.16 (VCC), U12.16 (VCC), U13.16 (VCC), U14.16 (VCC), U15.16 (VCC), U16.16 (VCC), U17.16 (VCC), U18.16 (VCC), U2.16 (VCC), U24.3 (Vin), U25.1 (A), U27.A4B9 (VBUS), U27.B4A9 (VBUS), U3.16 (VCC), U32.16 (+VO), U4.16 (VCC), U5.16 (VCC), U6.16 (VCC), U7.16 (VCC), U8.16 (VCC), U9.16 (VCC)
- net D+: now also R257.1, U28.47 (USB_DP); no longer R267.2
- net D-: now also U28.46 (USB_DM); no longer R268.2
- net GND: now also C40.2, R259.2, C31.1, C32.1, C33.2, C34.1, C35.1, C41.2, C42.2, C43.2, C44.2, C45.2, C46.2, C47.2, C48.2, C49.2, C50.2, C51.1, C52.1, D1.1, R254.1, R260.1, U1.13 (OE#), U1.8 (GND), U10.13 (OE#), U10.8 (GND), U11.13 (OE#), U11.8 (GND), U12.13 (OE#), U12.8 (GND), U13.13 (OE#), U13.8 (GND), U14.13 (OE#), U14.8 (GND), U15.13 (OE#), U15.8 (GND), U16.13 (OE#), U16.8 (GND), U17.13 (OE#), U17.8 (GND), U18.13 (OE#), U18.8 (GND), U19.2 (K), U2.13 (OE#), U2.8 (GND), U20.2 (K), U21.2 (K), U22.2 (K), U24.1 (GND), U27.13 (EH), U27.14 (EH), U27.A1B12 (GND), U27.B1A12 (GND), U28.19 (TESTEN), U28.57 (GND), U29.1 (A), U29.2 (B), U3.13 (OE#), U3.8 (GND), U30.1 (A), U30.2 (B), U31.2 (-), U32.14 (-VO), U33.4 (GND), U34.2 (E), U35.2 (E), U36.2 (E), U37.2 (E), U38.2 (E), U39.2 (E), U4.13 (OE#), U4.8 (GND), U40.2 (E), U41.2 (E), U5.13 (OE#), U5.8 (GND), U6.13 (OE#), U6.8 (GND), U7.13 (OE#), U7.8 (GND), U8.13 (OE#), U8.8 (GND), U9.13 (OE#), U9.8 (GND), X1.2 (GND), X1.4 (GND); no longer C40.1
- net POW: now also U31.3 (C2), U32.1 (AC/L)
- net VCOM: now also U31.4 (C1), U32.3 (AC/N); no longer NE2.2 (K)
- net XIN: now also C34.2, U28.20 (XIN), X1.1 (OSC1)
- net XOUT: now also R261.1, U28.21 (XOUT)
- net at R201.2: now also U12.10 (MR#)
- net at R218.2: now also U12.11 (SHCP)
- net at R236.2: now also U12.12 (STCP)
- net at R60.1: now also U2.3 (Q3)
- net at R100.1: now also U7.3 (Q3)
- net at R153.1: now also U14.15 (Q0)
- net at R65.1: now also U3.15 (Q0)
- net at R196.2: now also U22.1 (A)
- net at R231.2: now also U18.10 (MR#)
- net at R249.2: now also U18.11 (SHCP)
- net at R250.2: now also U18.12 (STCP)
- net at R63.1: now also U2.6 (Q6)
- net at R210.2: now also U2.10 (MR#)
- net at R227.2: now also U2.11 (SHCP)
- net at R245.2: now also U2.12 (STCP)
- net D_GPIO-2: now reaches R194.1, R232.1, R233.1, R234.1, R235.1, R236.1, R237.1, R238.1, R239.1, R240.1, R241.1, R242.1, R243.1, R244.1, R245.1, R246.1, R247.1, R248.1, R250.1
- net D_GPIO-2: now also U28.4 (GPIO2)
- net at R241.2: now also U4.12 (STCP)
- net at R49.1: now also U1.15 (Q0)
- net D_GPIO-0: now reaches R196.1, R197.1, R198.1, R199.1, R200.1, R201.1, R202.1, R203.1, R204.1, R205.1, R206.1, R207.1, R208.1, R209.1, R210.1, R211.1, R212.1, R213.1, R231.1
- net D_GPIO-0: now also U28.2 (GPIO0)
- net at R180.1: now also U17.3 (Q3)
- net at R179.1: now also U17.2 (Q2)
- net at R178.1: now also U17.1 (Q1)
- net at R177.1: now also U17.15 (Q0)
- net at R176.1: now also U16.7 (Q7)
- net at R175.1: now also U16.6 (Q6)
- net at R101.1: now also U7.4 (Q4)
- net D_GPIO-3: now reaches R193.1, R251.1
- net D_GPIO-3: now also U28.5 (GPIO3)
- net at R251.2: now also U1.14 (DS)
- net at R131.1: now also U11.2 (Q2)
- net at R156.1: now also U14.3 (Q3)
- net at R238.2: now also U3.12 (STCP)
- net at R91.1: now also U6.2 (Q2)
- net D_GPIO-1: now reaches R195.1, R214.1, R215.1, R216.1, R217.1, R218.1, R219.1, R220.1, R221.1, R222.1, R223.1, R224.1, R225.1, R226.1, R227.1, R228.1, R229.1, R230.1, R249.1
- net D_GPIO-1: now also U28.3 (GPIO1)
- net at R199.2: now also U13.10 (MR#)
- net at R216.2: now also U13.11 (SHCP)
- net at R234.2: now also U13.12 (STCP)
- net at R247.2: now also U10.12 (STCP)
- net at R150.1: now also U13.5 (Q5)
- net at R149.1: now also U13.4 (Q4)
- net at R148.1: now also U13.3 (Q3)
- net at R147.1: now also U13.2 (Q2)
- net at R146.1: now also U13.1 (Q1)
- net at R145.1: now also U13.15 (Q0)
- net at R169.1: now also U16.15 (Q0)
- net at R186.1: now also U18.1 (Q1)
- net at R185.1: now also U18.15 (Q0)
- net at R184.1: now also U17.7 (Q7)
- net at R183.1: now also U17.6 (Q6)
- net at R182.1: now also U17.5 (Q5)
- net at R181.1: now also U17.4 (Q4)
- net at R143.1: now also U12.6 (Q6)
- net at R76.1: now also U4.3 (Q3)
- net at R114.1: now also U9.1 (Q1)
- net at R113.1: now also U9.15 (Q0)
- net at R112.1: now also U8.7 (Q7)
- net at R111.1: now also U8.6 (Q6)
- net at R110.1: now also U8.5 (Q5)
- net at R109.1: now also U8.4 (Q4)
- net at R122.1: now also U10.1 (Q1)
- net at R198.2: now also U17.10 (MR#)
- net at R215.2: now also U17.11 (SHCP)
- net at R233.2: now also U17.12 (STCP)
- net at R136.1: now also U11.7 (Q7)
- net at R220.2: now also U3.11 (SHCP)
- net at R257.2: now also U27.A6 (Dp1), U27.B6 (Dp2)
- net at R59.1: now also U2.2 (Q2)
- net at R58.1: now also U2.1 (Q1)
- net at R57.1: now also U2.15 (Q0)
- net at R56.1: now also U1.7 (Q7)
- net at R55.1: now also U1.6 (Q6)
- net at R222.2: now also U1.11 (SHCP)
- net at R211.2: now also U7.10 (MR#)
- net at R258.2: now also U27.A7 (Dn1), U27.B7 (Dn2)
- net at R205.2: now also U1.10 (MR#)
- net at R161.1: now also U15.15 (Q0)
- net at R81.1: now also U5.15 (Q0)
- net at R84.1: now also U5.3 (Q3)
- net at R83.1: now also U5.2 (Q2)
- net at R82.1: now also U5.1 (Q1)
- net at R80.1: now also U4.7 (Q7)
- net at R79.1: now also U4.6 (Q6)
- net at R206.2: now also U4.10 (MR#)
- net at R268.1: now also U35.1 (B)
- net at R61.1: now also U2.4 (Q4)
- net at R68.1: now also U3.3 (Q3)
- net at R106.1: now also U8.1 (Q1)
- net at R135.1: now also U11.6 (Q6)
- net at R151.1: now also U13.6 (Q6)
- net at R73.1: now also U4.15 (Q0)
- net at R239.2: now also U5.12 (STCP)
- net at R130.1: now also U11.1 (Q1)
- net at R187.1: now also U18.2 (Q2)
- net at R223.2: now also U4.11 (SHCP)
- net at R96.1: now also U6.7 (Q7)
- net at R95.1: now also U6.6 (Q6)
- net at R94.1: now also U6.5 (Q5)
- net at R93.1: now also U6.4 (Q4)
- net at R92.1: now also U6.3 (Q3)
- net at R119.1: now also U9.6 (Q6)
- net D_GPIO-5: now reaches R269.2
- net D_GPIO-5: now also R267.2, U28.7 (GPIO5); no longer C40.2
- net at R105.1: now also U8.15 (Q0)
- net at R53.1: now also U1.4 (Q4)
- net at R90.1: now also U6.1 (Q1)
- net at R78.1: now also U4.5 (Q5)
- net at R144.1: now also U12.7 (Q7)
- net FLIP_32kHz_0B: now reaches R267.1
- net FLIP_32kHz_0B: now also R268.2, R270.1, U34.3 (C)
- net at R120.1: now also U9.7 (Q7)
- net at R118.1: now also U9.5 (Q5)
- net at R117.1: now also U9.4 (Q4)
- net at R116.1: now also U9.3 (Q3)
- net at R115.1: now also U9.2 (Q2)
- net at NE2.1 (A): now also R272.1, U37.3 (C); no longer R256.2
- net at R107.1: now also U8.2 (Q2)
- net at R214.2: now also U15.11 (SHCP)
- net at R237.2: now also U14.12 (STCP)
- net at R170.1: now also U16.1 (Q1)
- net at R224.2: now also U6.11 (SHCP)
- net at R155.1: now also U14.2 (Q2)
- net at R209.2: now also U11.10 (MR#)
- net at R203.2: now also U3.10 (MR#)
- net at R194.2: now also U20.1 (A)
- net at R152.1: now also U13.7 (Q7)
- net at R72.1: now also U3.7 (Q7)
- net at R71.1: now also U3.6 (Q6)
- net at R70.1: now also U3.5 (Q5)
- net at R69.1: now also U3.4 (Q4)
- net at R67.1: now also U3.2 (Q2)
- net at R197.2: now also U15.10 (MR#)
- net at R217.2: now also U16.11 (SHCP)
- net at R86.1: now also U5.5 (Q5)
- net at R158.1: now also U14.5 (Q5)
- net at R66.1: now also U3.1 (Q1)
- net at R64.1: now also U2.7 (Q7)
- net at R62.1: now also U2.5 (Q5)
- net at R132.1: now also U11.3 (Q3)
- net at R226.2: now also U11.11 (SHCP)
- net at R259.1: now also U25.2 (K)
- net at R188.1: now also U18.3 (Q3)
- net at R141.1: now also U12.4 (Q4)
- net at R193.2: now also U19.1 (A)
- net at R168.1: now also U15.7 (Q7)
- net at R192.1: now also U18.7 (Q7)
- net at R191.1: now also U18.6 (Q6)
- net at R190.1: now also U18.5 (Q5)
- net at R189.1: now also U18.4 (Q4)
- net at R134.1: now also U11.5 (Q5)
- net at R204.2: now also U5.10 (MR#)
- net at R54.1: now also U1.5 (Q5)
- net at R52.1: now also U1.3 (Q3)
- net at R51.1: now also U1.2 (Q2)
- net at R50.1: now also U1.1 (Q1)
- net at R171.1: now also U16.2 (Q2)
- net at R128.1: now also U10.7 (Q7)
- net at R138.1: now also U12.1 (Q1)
- net at R137.1: now also U12.15 (Q0)
- net at R133.1: now also U11.4 (Q4)
- net at R121.1: now also U10.15 (Q0)
- net at R139.1: now also U12.2 (Q2)
- net at R174.1: now also U16.5 (Q5)
- net at R173.1: now also U16.4 (Q4)
- net at R172.1: now also U16.3 (Q3)
- net at R208.2: now also U9.10 (MR#)
- net at R126.1: now also U10.5 (Q5)
- net at R125.1: now also U10.4 (Q4)
- net at R124.1: now also U10.3 (Q3)
- net at R123.1: now also U10.2 (Q2)
- net at R200.2: now also U16.10 (MR#)
- net at R154.1: now also U14.1 (Q1)
- net at R212.2: now also U10.10 (MR#)
- net at R229.2: now also U10.11 (SHCP)
- net at R77.1: now also U4.4 (Q4)
- net at R88.1: now also U5.7 (Q7)
- net at R104.1: now also U7.7 (Q7)
- net at R85.1: now also U5.4 (Q4)
- net at R213.2: now also U8.10 (MR#)
- net at R225.2: now also U9.11 (SHCP)
- net at R195.2: now also U21.1 (A)
- net at R221.2: now also U5.11 (SHCP)
- net at R89.1: now also U6.15 (Q0)
- net at R87.1: now also U5.6 (Q6)
- net at R228.2: now also U7.11 (SHCP)
- net at R108.1: now also U8.3 (Q3)
- net at R103.1: now also U7.6 (Q6)
- net at R232.2: now also U15.12 (STCP)
- net at R163.1: now also U15.2 (Q2)
- net at R166.1: now also U15.5 (Q5)
- net at R74.1: now also U4.1 (Q1)
- net at R246.2: now also U7.12 (STCP)
- net at R242.2: now also U6.12 (STCP)
- net at R167.1: now also U15.6 (Q6)
- net at R165.1: now also U15.4 (Q4)
- net at R164.1: now also U15.3 (Q3)
- net at R243.2: now also U9.12 (STCP)
- net at R142.1: now also U12.5 (Q5)
- net at R140.1: now also U12.3 (Q3)
- net at R97.1: now also U7.15 (Q0)
- net at R102.1: now also U7.5 (Q5)
- net at R230.2: now also U8.11 (SHCP)
- net at R75.1: now also U4.2 (Q2)
- net at R99.1: now also U7.2 (Q2)
- net at R98.1: now also U7.1 (Q1)
- net at R162.1: now also U15.1 (Q1)
- net at R160.1: now also U14.7 (Q7)
- net at R159.1: now also U14.6 (Q6)
- net at R157.1: now also U14.4 (Q4)
- net at R240.2: now also U1.12 (STCP)
- net at R235.2: now also U16.12 (STCP)
- net at R202.2: now also U14.10 (MR#)
- net at R219.2: now also U14.11 (SHCP)
- net at R129.1: now also U11.15 (Q0)
- net at R127.1: now also U10.6 (Q6)
- net at R207.2: now also U6.10 (MR#)
- net at R248.2: now also U8.12 (STCP)
- net at R244.2: now also U11.12 (STCP)
- new net: U1.9 (Q7S), U2.14 (DS)
- new net: U2.9 (Q7S), U3.14 (DS)
- new net: NE1.2 (K), R252.2, U40.3 (C)
- new net: U10.9 (Q7S), U11.14 (DS)
- new net: U11.9 (Q7S), U12.14 (DS)
- new net: R270.2, U36.1 (B)
- new net: NE2.2 (K), R255.1, U36.3 (C)
- new net: R266.1, U34.1 (B)
- new net: R263.2, U29.3 (C), U29.4 (D)
- new net: R260.2, U27.B5 (CC2)
- new net: U10.14 (DS), U9.9 (Q7S)
- new net: U7.9 (Q7S), U8.14 (DS)
- new net: U8.9 (Q7S), U9.14 (DS)
- new net: R271.2, U37.1 (B)
- new net: U6.9 (Q7S), U7.14 (DS)
- new net: U5.9 (Q7S), U6.14 (DS)
- new net: R273.1, U38.1 (B)
- new net: U14.9 (Q7S), U15.14 (DS)
- new net: U15.9 (Q7S), U16.14 (DS)
- new net: R274.1, U39.1 (B)
- new net: C33.1, R261.2, X1.3 (OSC2)
- new net: U13.9 (Q7S), U14.14 (DS)
- new net: R254.2, U27.A5 (CC1)
- new net: NE1.1 (A), R256.2, U41.3 (C)
- new net: U16.9 (Q7S), U17.14 (DS)
- new net: U17.9 (Q7S), U18.14 (DS)
- new net: U3.9 (Q7S), U4.14 (DS)
- new net: J1.1 (Pin_1), U28.25 (SWD)
- new net: J1.2 (Pin_2), U28.24 (SWCLK)
- new net: U12.9 (Q7S), U13.14 (DS)
- new net: U4.9 (Q7S), U5.14 (DS)
- new net: R277.2, U40.1 (B)
- new net: R278.2, U41.1 (B)
- new net: C37.1, R265.2, U28.43 (ADC_AVDD)
- new net +1V1: C46.1, C47.1, C48.1, U28.23 (DVDD), U28.45 (VREG_VOUT), U28.50 (DVDD)
- new net A_GPIO-26: U28.38 (GPIO26_ADC0)
- new net A_GPIO-27: U28.39 (GPIO27_ADC1)
- new net A_GPIO-28: U28.40 (GPIO28_ADC2)
- new net A_GPIO-29: U28.41 (GPIO29_ADC3)
- new net BOOT: R263.1, U28.56 (QSPI_SS), U33.1 (CS#)
- new net D_GPIO-10: U28.13 (GPIO10)
- new net D_GPIO-11: U28.14 (GPIO11)
- new net D_GPIO-12: U28.15 (GPIO12)
- new net D_GPIO-13: U28.16 (GPIO13)
- new net D_GPIO-14: U28.17 (GPIO14)
- new net D_GPIO-15: U28.18 (GPIO15)
- new net D_GPIO-16: U28.27 (GPIO16)
- new net D_GPIO-17: U28.28 (GPIO17)
- new net D_GPIO-18: U28.29 (GPIO18)
- new net D_GPIO-19: U28.30 (GPIO19)
- new net D_GPIO-20: U28.31 (GPIO20)
- new net D_GPIO-21: U28.32 (GPIO21)
- new net D_GPIO-22: U28.34 (GPIO22)
- new net D_GPIO-23: U28.35 (GPIO23)
- new net D_GPIO-24: U28.36 (GPIO24)
- new net D_GPIO-25: U28.37 (GPIO25)
- new net D_GPIO-4: R275.2, R276.2, U28.6 (GPIO4)
- new net D_GPIO-6: U28.8 (GPIO6)
- new net D_GPIO-7: U28.9 (GPIO7)
- new net D_GPIO-8: U28.11 (GPIO8)
- new net D_GPIO-9: U28.12 (GPIO9)
- new net FLIP_32kHz: C50.1, R266.2, R273.2, TXAL1.2
- new net FLIP_32kHz_0A: R274.2, R275.1, R277.1, U38.3 (C)
- new net FLIP_32kHz_1A: R276.1, R278.1, U39.3 (C)
- new net FLIP_32kHz_1B: R269.1, R271.1, U35.3 (C)
- new net MEM_CLK: U28.52 (QSPI_SCLK), U33.6 (CLK)
- new net MEM_DI: U28.53 (QSPI_SD0), U33.5 (DI)
- new net MEM_DO: U28.55 (QSPI_SD1), U33.2 (DO)
- new net ~{MEM_HOLD}: U28.51 (QSPI_SD3), U33.7 (IO3)
- new net ~{MEM_WP}: U28.54 (QSPI_SD2), U33.3 (IO2)
- new net ~{RESET}: U28.26 (RUN), U30.3 (C), U30.4 (D)
Other:
- note added: "Latch Clock"
- note added: "Serial"
- note added: "Serial Clock"
- note added: "~{Reset}"
- moved on the sheet: F1, NX1, NX10, NX11, NX12, NX2, NX3, NX4, NX5, NX6, NX7, NX8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

Commit message: Final changes before printing
Parts:
- removed C49, C50: 15pF, Capacitor_SMD:C_0402_1005Metric, symbol NixMinis:Mini_C
- removed TXAL1: Q13FC1350000400, JLCPCB_Imported:FC-135R_L3.2-W1.5, symbol JLCPCB_Imported:Q13FC1350000400
- F1, U32: now not fitted
- SW1: now not fitted; now left out of the parts list
Connections:
- net FLIP_32kHz is gone; now on net D_GPIO-6: R266.2, R273.2
